Commit message: Human urdf fixed

File: urdf/human.urdf (robot description, URDF)
Before this commit: robot human_xacro, 28 links, 27 joints
Links:
- added link front_left_steer_link, mass 1; collision cylinder length=0.4 radius=0.03; visual cylinder length=0.4 radius=0.03
- added link front_right_steer_link, mass 1; collision cylinder length=0.4 radius=0.03; visual cylinder length=0.4 radius=0.03
- added link rear_left_steer_link, mass 1; collision cylinder length=0.4 radius=0.03; visual cylinder length=0.4 radius=0.03
- added link rear_right_steer_link, mass 1; collision cylinder length=0.4 radius=0.03; visual cylinder length=0.4 radius=0.03
- link back_link: geometry collision box size=0.4 0.4 0.04; visual box size=0.5 0.4 0.04
- link base_link: geometry collision box size=0.4 0.4 0.04; visual box size=0.4 0.4 0.04
- link body_link: geometry collision box size=0.5 0.25 0.1; visual box size=0.5 0.25 0.1
- link bodyleft_link: geometry collision cylinder length=0.5 radius=0.05; visual cylinder length=0.5 radius=0.05
- link bodyright_link: geometry collision cylinder length=0.5 radius=0.05; visual cylinder length=0.5 radius=0.05
- link panelback_link: geometry collision box size=0.8 0.3 0.02; visual box size=0.8 0.3 0.02
- link panelfront_link: geometry collision box size=0.8 0.3 0.02; visual box size=0.8 0.3 0.02
Joints:
- added joint front_left_steer_joint: type revolute, parent base_link, child front_left_steer_link, origin xyz=0.15 -0.15 -0.4 rpy=0 0 0, axis 0 0 1, limit lower=-3.14159265359 upper=3.14159265359 effort=10.0 velocity=5.0
- added joint front_right_steer_joint: type revolute, parent base_link, child front_right_steer_link, origin xyz=0.15 0.15 -0.4 rpy=0 0 0, axis 0 0 1, limit lower=-3.14159265359 upper=3.14159265359 effort=10.0 velocity=5.0
- added joint rear_left_steer_joint: type revolute, parent base_link, child rear_left_steer_link, origin xyz=-0.15 -0.15 -0.4 rpy=0 0 0, axis 0 0 1, limit lower=-3.14159265359 upper=3.14159265359 effort=10.0 velocity=5.0
- added joint rear_right_steer_joint: type revolute, parent base_link, child rear_right_steer_link, origin xyz=-0.15 0.15 -0.4 rpy=0 0 0, axis 0 0 1, limit lower=-3.14159265359 upper=3.14159265359 effort=10.0 velocity=5.0
- joint armleft2_armleft3_joint: origin xyz=-0.065 0 0.11 rpy=0 ${-30 * deg_to_rad} 0 -> xyz=-0.065 0 0.11 rpy=0 -0.523598775598 0
- joint armleft3_handleft_joint: origin xyz=0 0 ${0.2*0.5} rpy=0 0 0 -> xyz=0 0 0.1 rpy=0 0 0
- joint armrighht3_handright_joint: origin xyz=0 0 ${0.2*0.5} rpy=0 0 0 -> xyz=0 0 0.1 rpy=0 0 0
- joint armright2_armright3_joint: origin xyz=-0.065 0 0.11 rpy=0 ${-30 * deg_to_rad} 0 -> xyz=-0.065 0 0.11 rpy=0 -0.523598775598 0
- joint base_back_joint: origin xyz=${-length/2.0 + 0.02} 0 ${length/2.0} rpy=0 ${-90 * deg_to_rad} 0 -> xyz=-0.18 0 0.2 rpy=0 -1.57079632679 0
- joint base_body_joint: origin xyz=-0.0 0 ${human_back_length/2.0} rpy=0 ${-90 * deg_to_rad} 0 -> xyz=-0.0 0 0.25 rpy=0 -1.57079632679 0
- joint base_footprint_joint: origin xyz=0 0 ${wheel_radius} rpy=0 0 0 -> xyz=0 0 0.11 rpy=0 0 0
- joint base_panelback_joint: origin xyz=-0.08 0.45 -0.005 rpy=0 ${-80 * deg_to_rad} 0 -> xyz=-0.08 0.45 -0.005 rpy=0 -1.3962634016 0
- joint base_panelfront_joint: origin xyz=0.08 0.45 -0.005 rpy=0 ${80 * deg_to_rad} 0 -> xyz=0.08 0.45 -0.005 rpy=0 1.3962634016 0
- joint body_bodyleft_joint: origin xyz=0.0 0.125 0 rpy=0 ${-90 * deg_to_rad} 0 -> xyz=0.0 0.125 0 rpy=0 -1.57079632679 0
- joint body_bodyright_joint: origin xyz=0.0 -0.125 0 rpy=0 ${-90 * deg_to_rad} 0 -> xyz=0.0 -0.125 0 rpy=0 -1.57079632679 0
- joint body_chest_joint: origin xyz=0.25 0 0 rpy=${-90 * deg_to_rad} 0 0 -> xyz=0.25 0 0 rpy=-1.57079632679 0 0
- joint bodyleft_legleft1_joint: origin xyz=-0.2 0 ${human_back_length/2-0.075} rpy=0 ${-90 * deg_to_rad} 0 -> xyz=-0.2 0 0.175 rpy=0 -1.57079632679 0
- joint bodyright_legright1_joint: origin xyz=-0.2 0 ${human_back_length/2-0.075} rpy=0 ${-90 * deg_to_rad} 0 -> xyz=-0.2 0 0.175 rpy=0 -1.57079632679 0
- joint legleft2_legleft3_joint: origin xyz=0.225 0 0 rpy=0 ${-90 * deg_to_rad} 0 -> xyz=0.225 0 0 rpy=0 -1.57079632679 0
- joint legleft3_footleft_joint: origin xyz=0.05 0 -${0.45*0.5} rpy=0 0 0 -> xyz=0.05 0 -0.225 rpy=0 0 0
- joint legright2_legright3_joint: origin xyz=0.225 0 0 rpy=0 ${-90 * deg_to_rad} 0 -> xyz=0.225 0 0 rpy=0 -1.57079632679 0
- joint legrihgt3_footrihgt_joint: origin xyz=0.05 0 -${0.45*0.5} rpy=0 0 0 -> xyz=0.05 0 -0.225 rpy=0 0 0
- joint shoulderleft_armleft1_joint: origin xyz=-0.065 0 0.11 rpy=0 ${-30 * deg_to_rad} 0 -> xyz=-0.065 0 0.11 rpy=0 -0.523598775598 0
- joint shoulderright_armright1_joint: origin xyz=-0.065 0 0.11 rpy=0 ${-30 * deg_to_rad} 0 -> xyz=-0.065 0 0.11 rpy=0 -0.523598775598 0
