Commit message: Robot Model as Dog + Materials + gazebo file

File: urdf/robot.xacro (robot description, xacro)
@@ -2,43 +2,87 @@
 <robot xmlns:xacro="http://www.ros.org/wiki/xacro" name="robot_xacro">
 <xacro:include filename="$(find exp_assignment2)/urdf/robot.gazebo"/>
-	<xacro:property name="length_wheel" value="0.04" />
-	<xacro:property name="radius_wheel" value="0.1" />
-	<xacro:macro name="default_inertial" params="mass">
-               <inertial>
-                       <mass value="${mass}" />
-                       <origin rpy="0 1.5707 1.5707" xyz="0 0 0"/>
-                       <inertia ixx="0.000526666666667" ixy="0" ixz="0" iyy="0.000526666666667" iyz="0" izz="0.001"/>
-               </inertial>
-	</xacro:macro>
-    <xacro:macro name="wheel_geometry">
-		<geometry>
-       			<cylinder length="${length_wheel}" radius="${radius_wheel}"/>
-     	</geometry>
-	</xacro:macro>
-  <material name="black">
-    <color rgba="0.0 0.0 0.0 1.0"/>
-  </material>
-  <material name="blue">
-    <color rgba="0.203125 0.23828125 0.28515625 1.0"/>
-  </material>
-  <material name="green">
-    <color rgba="0.0 0.8 0.0 1.0"/>
-  </material>
-  <material name="grey">
-    <color rgba="0.2 0.2 0.2 1.0"/>
-  </material>
-  <material name="orange">
-    <color rgba="1.0 0.423529411765 0.0392156862745 1.0"/>
-  </material>
-  <material name="brown">
-    <color rgba="0.870588235294 0.811764705882 0.764705882353 1.0"/>
-  </material>
-  <material name="red">
-    <color rgba="0.80078125 0.12890625 0.1328125 1.0"/>
-  </material>
-  <material name="white">
-    <color rgba="1.0 1.0 1.0 1.0"/>
-  </material>
-	  <link name="link_chassis">
+  <!-- materials -->
+<xacro:include filename="$(find exp_assignment2)/urdf/materials.xacro" />
+ <xacro:include filename="$(find exp_assignment2)/urdf/robot.gazebo" />
+ <xacro:property name="length_wheel" value="0.05" />
+ <xacro:property name="radius_wheel" value="0.15" />
+ <xacro:property name="neck_length" value="0.1" />
+ <xacro:property name="neck_radius" value="0.04" />
+ <xacro:property name="camera_link" value="0.05" /> <!-- Size of square 'camera' box -->
+ <xacro:macro name="cylinder_inertia" params="mass r l">
+    <inertia ixx="${mass*(3*r*r+l*l)/12}" ixy = "0" ixz = "0"
+                iyy="${mass*(3*r*r+l*l)/12}" iyz = "0" izz="${mass*(r*r)/2}" />
+ </xacro:macro>
+ <xacro:macro name="box_inertia" params="mass w h d">
+    <inertia ixx="${mass*(h*h+d*d)/12}" ixy = "0" ixz = "0"
+                iyy="${mass*(w*w+d*d)/12}" iyz = "0" izz="${mass*(w*w+h*h)/12}" />
+ </xacro:macro>
+ <xacro:macro name="link_ear" params="name">
+   <link name="${name}">
+            <inertial>
+              <mass value="0.1"/>
+              <origin rpy="0 0 0" xyz="0 0 0"/>
+              <!-- <inertia ixx="0.000526666666667" ixy="0" ixz="0" iyy="0.000526666666667" iyz="0" izz="0.001"/> -->
+	      <xacro:box_inertia mass="0.1" w="0.05" h="0.03" d="0.034"/>
+            </inertial>
+            <collision name="${name}_collision">
+              <origin rpy="0 0 1.5708" xyz="0 0 0"/>
+              <geometry>
+                <box size="0.034 0.05 0.03"/>
+              </geometry>
+            </collision>
+            <visual name="${name}_visual">
+              <origin rpy="0 0 0" xyz="0 0 0"/>
+              <geometry>
+                <box size="0.034 0.05 0.03"/>
+              </geometry>
+		<material name="blue" />
+            </visual>
+        </link>
+ </xacro:macro>
+    <xacro:macro name="joint_ear" params="name child origin_xyz">
+      <joint name="${name}" type="fixed">
+        <origin rpy="0 0 0" xyz="${origin_xyz}"/>
+        <child link="${child}"/>
+        <parent link="head_link"/>
+        <axis rpy="0 0 0" xyz="0 0 1"/>
+        <limit effort="10000" velocity="1000"/>
+        <joint_properties damping="1.0" friction="1.0"/>
+      </joint>
+    </xacro:macro>
+    <xacro:macro name="link_wheel" params="name">
+        <link name="${name}">
+            <inertial>
+              <mass value="0.2"/>
+              <origin rpy="0 1.5707 1.5707" xyz="0 0 0"/>
+              <!-- <inertia ixx="0.000526666666667" ixy="0" ixz="0" iyy="0.000526666666667" iyz="0" izz="0.001"/> -->
+	      <xacro:cylinder_inertia mass="0.2" r="${radius_wheel}" l="${length_wheel}" />
+            </inertial>
+            <collision name="link_right_wheel_collision">
+              <origin rpy="0 1.5707 1.5707" xyz="0 0 0"/>
+              <geometry>
+                <cylinder length="${length_wheel}" radius="${radius_wheel}"/>
+              </geometry>
+            </collision>
+            <visual name="${name}_visual">
+              <origin rpy="0 1.5707 1.5707" xyz="0 0 0"/>
+              <geometry>
+                <cylinder length="${length_wheel}" radius="${radius_wheel}"/>
+              </geometry>
+            </visual>
+        </link>
+    </xacro:macro>
+    <xacro:macro name="joint_wheel" params="name child origin_xyz">
+      <joint name="${name}" type="continuous">
+        <origin rpy="0 0 0" xyz="${origin_xyz}"/>
+        <child link="${child}"/>
+        <parent link="base_link"/>
+        <axis rpy="0 0 0" xyz="0 1 0"/>
+        <limit effort="10000" velocity="1000"/>
+        <joint_properties damping="1.0" friction="1.0"/>
+      </joint>
+    </xacro:macro>
+<!-- _______________base link____________________  -->
+  <link name="base_link">
     <!-- pose and inertial -->
     <pose>0 0 0.1 0 0 0</pose>
@@ -48,5 +92,4 @@
       <inertia ixx="0.0395416666667" ixy="0" ixz="0" iyy="0.106208333333" iyz="0" izz="0.106208333333"/>
     </inertial>
-    <!-- body -->
     <collision name="collision_chassis">
       <geometry>
@@ -67,4 +110,14 @@
         <sphere radius="0.05"/>
       </geometry>
+      <surface>
+        <friction>
+          <ode>
+            <mu>0</mu>
+            <mu2>0</mu2>
+            <slip1>1.0</slip1>
+            <slip2>1.0</slip2>
+          </ode>
+        </friction>
+      </surface>
     </collision>
     <visual name="caster_front_visual">
@@ -74,72 +127,109 @@
       </geometry>
     </visual>
+    </link>
+  <!-- Create wheels -->
+  <xacro:link_wheel name="link_right_wheel" />
+  <xacro:link_wheel name="link_left_wheel" />
+  <xacro:joint_wheel name="joint_right_wheel"  child="link_right_wheel"  origin_xyz="-0.05 0.15 0"  />
+  <xacro:joint_wheel name="joint_left_wheel"   child="link_left_wheel"   origin_xyz="-0.05 -0.15 0"  />
+<!-- _______________neck definition_______________ -->
+  <link name="neck_link">
+  	<inertial>
+  		<mass value="0.025"/>
+  		<origin xyz="0 0 0" rpy="0 0 0" />
+  		<!--<inertia ixx="0.000010279" ixy="0" ixz="0" iyy="0.000010279" iyz="0" izz="0.000007225"/>-->
+		<xacro:cylinder_inertia mass="0.2" r="${neck_radius}" l="${neck_length}" />
+  	</inertial>
+  	<collision>
+  	  <origin xyz="0 0 ${neck_length/2}" rpy="0 0 0"/> <!-- frame moved to the base of the cylinder -->
+      <geometry>
+        <cylinder radius="${neck_radius}" length="${neck_length}"/>
+      </geometry>
+  	</collision>
+  	<visual>
+  	  <origin xyz="0 0 ${neck_length/2}" rpy="0 0 0"/> <!-- frame moved to the base of the cylinder -->
+      <geometry>
+        <cylinder radius="${neck_radius}" length="${neck_length}"/>
+      </geometry>
+      <material name="red" />
+  	</visual>
   </link>
-   <link name="link_right_wheel">
-    <xacro:default_inertial mass="0.2"/>
-    <collision name="link_right_wheel_collision">
-      <origin rpy="0 1.5707 1.5707" xyz="0 0 0"/>
-      <xacro:wheel_geometry />
+  <joint name="neck_joint" type="fixed">
+  	<axis xyz="0 0 1"/>
+  	<limit effort="1000.0" lower="-3.14" upper="3.14" velocity="0.2"/>
+  	<origin rpy="0 0 0" xyz="0.15 0 0.035"/> <!-- half the height of the base link -->
+  	<parent link="base_link"/>
+  	<child link="neck_link"/>
+  </joint>
+<!-- head definition -->
+    <link name="head_link">
+  	<inertial>
+  		<mass value="0.025"/>
+  		<origin xyz="0 0 0" rpy="0 0 0" />
+  		<xacro:box_inertia mass="0.025" w="0.2" h="0.08" d="0.034"/>
+  	</inertial>
+  	<collision>
+  	  <origin xyz="0 0 0.04" rpy="0 0 0"/> <!-- frame moved to the base of the head -->
+      <geometry>
+        <box size="0.034 0.2 0.08"/>
+      </geometry>
+  	</collision>
+  	<visual>
+  	  <origin xyz="0 0 0.04" rpy="0 0 0"/> <!-- frame moved to the base of the head -->
+      <geometry>
+        <box size="0.034 0.2 0.08"/>
+      </geometry>
+      <material name="red" />
+  	</visual>
+  </link>
+  <joint name="head_joint" type="revolute">
+  	<axis xyz="0 0 1"/>
+  	<limit effort="1000.0" lower="-1.8" upper="1.8" velocity="0.5"/>
+  	<origin rpy="0 0 0" xyz="0 0 ${neck_length}"/>
+  	<parent link="neck_link"/>
+  	<child link="head_link"/>
+  </joint>
+ <!-- Camera -->
+  <link name="camera_link">
+    <collision>
+      <origin xyz="0 0 0" rpy="0 0 0"/>
+      <geometry>
+    <box size="${camera_link} ${camera_link} ${camera_link}"/>
+      </geometry>
     </collision>
-    <visual name="link_right_wheel_visual">
-      <origin rpy="0 1.5707 1.5707" xyz="0 0 0"/>
-      <xacro:wheel_geometry />
+    <visual>
+      <origin xyz="0 0 0" rpy="0 0 0"/>
+      <geometry>
+    <box size="${camera_link} ${camera_link} ${camera_link}"/>
+      </geometry>
       <material name="red"/>
     </visual>
-  </link>
-   <link name="link_left_wheel">
-    <xacro:default_inertial mass="0.2"/>
-    <collision name="link_left_wheel_collision">
-      <origin rpy="0 1.5707 1.5707" xyz="0 0 0"/>
-      <xacro:wheel_geometry />
-    </collision>
-    <visual name="link_left_wheel_visual">
-      <origin rpy="0 1.5707 1.5707" xyz="0 0 0"/>
-      <xacro:wheel_geometry />
-      <material name="red"/>
-    </visual>
-  </link>
-  <joint name="joint_right_wheel" type="continuous">
-    <origin rpy="0 0 0" xyz="-0.05 0.15 0"/>
-    <child link="link_right_wheel"/>
-    <parent link="link_chassis"/>
-    <axis rpy="0 0 0" xyz="0 1 0"/>
-    <limit effort="10000" velocity="1000"/>
-    <joint_properties damping="1.0" friction="1.0"/>
-  </joint>
-  <joint name="joint_left_wheel" type="continuous">
-    <origin rpy="0 0 0" xyz="-0.05 -0.15 0"/>
-    <child link="link_left_wheel"/>
-    <parent link="link_chassis"/>
-    <axis rpy="0 0 0" xyz="0 1 0"/>
-    <limit effort="10000" velocity="1000"/>
-    <joint_properties damping="1.0" friction="1.0"/>
-  </joint>
-  <link name="camera_link">
-	    <collision>
-	      <origin xyz="0 0 0.025" rpy="0 0 0"/>
-	      <geometry>
-		<box size="0.05 0.05 0.05"/>
-	      </geometry>
-	    </collision>
-	    <visual>
-	      <origin xyz="0 0 0.025" rpy="0 0 0"/>
-	      <geometry>
-		<box size="0.05 0.05 0.05"/>
-	      </geometry>
-	      <material name="red">
-		<color rgba="1 0 0 1"/>
-	      </material>
-	    </visual>
-	    <inertial>
-	      <mass value="1e-5" />
-	      <origin xyz="0 0 0" rpy="0 0 0"/>
-	      <inertia ixx="1e-6" ixy="0" ixz="0" iyy="1e-6" iyz="0" izz="1e-6" />
-	    </inertial>
+    <inertial>
+      <mass value="1e-5" />
+      <origin xyz="0 0 0" rpy="0 0 0"/>
+      <inertia ixx="1e-6" ixy="0" ixz="0" iyy="1e-6" iyz="0" izz="1e-6" />
+    </inertial>
   </link>
   <joint name="camera_joint" type="fixed">
-	    <axis xyz="0 1 0" />
-	    <origin xyz="0.23 0 0.0" rpy="0 0 0"/>
-	    <parent link="link_chassis"/>
-	    <child link="camera_link"/>
-	 </joint>
+    <axis xyz="0 1 0" />
+    <origin xyz="0 0.017 0.04" rpy="0 0 0"/>
+    <parent link="head_link"/>
+    <child link="camera_link"/>
+  </joint>
+<!-- hears definition -->
+  <xacro:link_ear name="link_right_ear" />
+  <xacro:link_ear name="link_left_ear" />
+  <xacro:joint_ear name="joint_right_ear"  child="link_right_ear"  origin_xyz="0 0.08 0.08"  />
+  <xacro:joint_ear name="joint_left_ear"   child="link_left_ear"   origin_xyz="0 -0.08 0.08"  />
+<!-- transmission -->
+<transmission name="head_joint_trans">
+	<type>transmission_interface/SimpleTransmission</type>
+	<joint name="head_joint">
+		<hardwareInterface>hardware_interface/EffortJointInterface</hardwareInterface>
+	</joint>
+	<actuator name="motor1">
+		<hardwareInterface>hardware_interface/EffortJointInterface</hardwareInterface>
+		<mechanicalInterface>1</mechanicalInterface>
+	</actuator>
+</transmission>
 </robot>

Commit message: implemented cmd_manager-py

File: urdf/robot.xacro (robot description, xacro)
@@ -5,12 +5,15 @@
 <xacro:include filename="$(find exp_assignment2)/urdf/materials.xacro" />
  <xacro:include filename="$(find exp_assignment2)/urdf/robot.gazebo" />
- <xacro:property name="length_wheel" value="0.05" />
- <xacro:property name="radius_wheel" value="0.15" />
+ <xacro:property name="length_wheel" value="0.04" />
+ <xacro:property name="radius_wheel" value="0.10" />
  <xacro:property name="neck_length" value="0.1" />
- <xacro:property name="neck_radius" value="0.04" />
+ <xacro:property name="neck_radius" value="0.03" />
  <xacro:property name="camera_link" value="0.05" /> <!-- Size of square 'camera' box -->
  <xacro:macro name="cylinder_inertia" params="mass r l">
     <inertia ixx="${mass*(3*r*r+l*l)/12}" ixy = "0" ixz = "0"
                 iyy="${mass*(3*r*r+l*l)/12}" iyz = "0" izz="${mass*(r*r)/2}" />
+ </xacro:macro>
+ <xacro:macro name="sphere_inertia" params="mass r">
+	<inertia ixx="${(mass*r*r)/4" ixy = "0" ixz = "0" iyy="${(mass*r*r)/4" iyx = "0" iyz  = "0" izz="${(mass*r*r)/2" />
  </xacro:macro>
  <xacro:macro name="box_inertia" params="mass w h d">
@@ -182,9 +185,9 @@
       <material name="red" />
   	</visual>
-  </link>
+</link>
   <joint name="head_joint" type="revolute">
   	<axis xyz="0 0 1"/>
   	<limit effort="1000.0" lower="-1.8" upper="1.8" velocity="0.5"/>
-  	<origin rpy="0 0 0" xyz="0 0 ${neck_length}"/>
+  	<origin rpy="0 0 0" xyz="0.15 0 ${neck_length}"/>
   	<parent link="neck_link"/>
   	<child link="head_link"/>

Commit message: Added behaviour for play state + fix some bugs in the scripts files

File: urdf/robot.xacro (robot description, xacro)
@@ -20,10 +20,10 @@
                 iyy="${mass*(w*w+d*d)/12}" iyz = "0" izz="${mass*(w*w+h*h)/12}" />
  </xacro:macro>
- <xacro:macro name="link_ear" params="name">
+ <!-- <xacro:macro name="link_ear" params="name">
    <link name="${name}">
             <inertial>
               <mass value="0.1"/>
               <origin rpy="0 0 0" xyz="0 0 0"/>
-              <!-- <inertia ixx="0.000526666666667" ixy="0" ixz="0" iyy="0.000526666666667" iyz="0" izz="0.001"/> -->
+              <inertia ixx="0.000526666666667" ixy="0" ixz="0" iyy="0.000526666666667" iyz="0" izz="0.001"/>
 	      <xacro:box_inertia mass="0.1" w="0.05" h="0.03" d="0.034"/>
             </inertial>
@@ -53,4 +53,5 @@
       </joint>
     </xacro:macro>
+-->
     <xacro:macro name="link_wheel" params="name">
         <link name="${name}">
@@ -188,5 +189,5 @@
   	<axis xyz="0 0 1"/>
   	<limit effort="1000.0" lower="-1.8" upper="1.8" velocity="0.5"/>
-  	<origin rpy="0 0 0" xyz="0.15 0 ${neck_length}"/>
+  	<origin rpy="0 0 0" xyz="0 0 ${neck_length}"/>
   	<parent link="neck_link"/>
   	<child link="head_link"/>
@@ -220,8 +221,8 @@
   </joint>
 <!-- hears definition -->
-  <xacro:link_ear name="link_right_ear" />
+  <!-- <xacro:link_ear name="link_right_ear" />
   <xacro:link_ear name="link_left_ear" />
   <xacro:joint_ear name="joint_right_ear"  child="link_right_ear"  origin_xyz="0 0.08 0.08"  />
-  <xacro:joint_ear name="joint_left_ear"   child="link_left_ear"   origin_xyz="0 -0.08 0.08"  />
+  <xacro:joint_ear name="joint_left_ear"   child="link_left_ear"   origin_xyz="0 -0.08 0.08"  /> -->
 <!-- transmission -->
 <transmission name="head_joint_trans">
